File: hardware/dynext_v1.1.brd (EAGLE design)
At the start: 32.5 x 17.8 mm, 44 parts, among them IC1 TPS560200, IC2 LM4040D20IDBZT, J1 AVR_SPI_PRG_6PTH, P1 PIN_SMD_2X2.5, P2 PIN_SMD_2X2.5, U1 ATxmega16E5, U2 TLV70033DCK, U4 TXB0101DCK, U5 TXB0101DCK, X1 CRYSTAL-0500290P1

Commit message: Cleanup of versions of the board. Added semi-corrected version of v1, it I ever want to go back to it...
Parts:
- removed C11: 0.1uF, Xevelabs:0402_N
- D1, D3, D4: device Xevelabs:SOD-523_N -> Xevelabs:SOD-923_N
- moved DXL2 5.06 mm to (2.50, 0.40), turned to 90 degrees
- moved DXL1 2.45 mm to (2.45, 17.9), turned to 90 degrees
Connections:
- removed net N$1: C11.1, DXL3.GND
- net +12V: now also DXL3.VBUS
- net GND: now also DXL3.GND; no longer C11.2
Routing:
- net +12V: track 13.5 -> 31.4 mm
- net GND: track 12.9 -> 18.4 mm, vias 17 -> 16
- net N$7: track 7.68 -> 4.21 mm
- net N$11: track 5.78 -> 2.44 mm
- net N$1: track 1.74 -> 0.00 mm
- net +5V: track 13.4 -> 11.8 mm
- net DATA: track 38.1 -> 38.9 mm
Other:
- board text added: "v1.1"
- board text removed: "Not fit for use as is. Errors: - SOT-523 diodes should be SOT-923 - DXL connectors are reversed"
- board text removed: "v1.0"
