File: hardware/dynext_v2.0.brd (EAGLE design)
At the start: 34.3 x 17.8 mm, 50 parts, among them IC1 TCR2EE50,LM, P1 PIN_SMD_0.8X2, P2 PIN_SMD_1X1, P3 PIN_SMD_0.8X2, P4 PIN_SMD_0.8X2, P5 PIN_SMD_0.8X2, P6 PIN_SMD_1X1, P7 PIN_SMD_1X1, U1 TPS62160DSG, U2 LD6805K/33P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

Commit message: Updated schematics with final values for the switch reg voltage divider.
Parts:
- R2: value todok 1% -> 1.02M 1%
- R3: value todok 1% -> 178k 1%
- Y1: value CSTCE16M0V53 -> CSTCE16M0V53-R0
Connections:
- net 5.25V renamed 5V_DIRTY
Changed lines of the file:
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@@
 <?xml version="1.0" encoding="utf-8"?>
 <!DOCTYPE eagle SYSTEM "eagle.dtd">
-<eagle version="6.4">
+<eagle version="6.5.0">
 <drawing>
 <settings>
@@
 <layer number="21" name="tPlace" color="7" fill="1" visible="no" active="yes"/>
 <layer number="22" name="bPlace" color="7" fill="1" visible="no" active="yes"/>
-<layer number="23" name="tOrigins" color="15" fill="1" visible="no" active="yes"/>
+<layer number="23" name="tOrigins" color="15" fill="1" visible="yes" active="yes"/>
 <layer number="24" name="bOrigins" color="15" fill="1" visible="no" active="yes"/>
 <layer number="25" name="tNames" color="7" fill="1" visible="no" active="yes"/>
@@
 <element name="U4" library="Xevelabs" package="SC70-6" value="TXB0101DCK" x="17.99" y="3.93" rot="R180"/>
 <element name="LED2" library="Xevelabs" package="D_0603_N" value="Red" x="25.09" y="1.12"/>
-<element name="R2" library="Xevelabs" package="0201_N" value="todok 1%" x="3.53" y="5.365" rot="R270"/>
-<element name="R3" library="Xevelabs" package="0201_N" value="todok 1%" x="3.53" y="6.895" rot="R90"/>
+<element name="R2" library="Xevelabs" package="0201_N" value="1.02M 1%" x="3.53" y="5.365" rot="R270"/>
+<element name="R3" library="Xevelabs" package="0201_N" value="178k 1%" x="3.53" y="6.895" rot="R90"/>
 <element name="C17" library="Xevelabs" package="1206_N" value="22uF" x="7.4" y="5.5" rot="R90"/>
 <element name="R1" library="Xevelabs" package="0201_N" value="1K" x="25.38" y="2.28"/>
@@
 </element>
 <element name="JP10" library="SparkFun-Connectors" package="1X05-1.27MM" value="SWD" x="19.035" y="7.92" rot="R180"/>
-<element name="Y1" library="SparkFun-FreqCtrl" package="RESONATOR-SMD" value="CSTCE16M0V53" x="16.495" y="10.65" rot="R180">
+<element name="Y1" library="SparkFun-FreqCtrl" package="RESONATOR-SMD" value="CSTCE16M0V53-R0" x="16.495" y="10.65" rot="R180">
 <attribute name="PROD_ID" value="XTAL-08900" x="16.495" y="10.65" size="1.778" layer="27" rot="R180" display="off"/>
 </element>
@@
 <wire x1="16.825" y1="8.86" x2="17.765" y2="7.92" width="0.15" layer="1"/>
 </signal>
-<signal name="5.25V">
+<signal name="5V_DIRTY">
 <contactref element="U1" pad="6"/>
 <contactref element="R2" pad="2"/>
