File: hardware/dynext_v2.0.sch (EAGLE design)
At the start: 40 parts, among them P1 PIN_SMD_2X2.5, P2 PIN_SMD_2X2.5, P3 PIN_SMD_0.8X2, P4 PIN_SMD_0.8X2, U2 LD6805K/33P, U3 IC_ATMEGA328P-MMH, U4 TXB0101DCK, U6 LPC11A02UK,118, Y1 CSTCE16M0V53

Commit message: Shifting things around, preparing for the real pinout & layout.
Parts:
- removed JP2: M09, SparkFun-Connectors:M09
- added C4: 1uF, Xevelabs:C0402
- added IC1: TCR2EE50,LM, Xevelabs:IC_TCR2EEESV
- JP1: device SparkFun-Connectors:M07 -> SparkFun-Connectors:M03PTH
Connections:
- net D13 renamed D13/LED
- removed net PA2: JP1.3
- removed net PA3: JP1.4
- removed net PA7: JP1.5
- removed net PC0: JP1.6
- removed net PC1: JP1.7
- removed net PC4: JP2.7
- removed net PC5: JP2.6
- removed net PC6: JP2.5
- removed net PC7: JP2.4
- net +3V3: now also C6.1, U2.OUT; no longer C14.1, JP1.2
- net +5V: now also C14.1, IC1.VOUT; no longer C6.1, JP2.2, U2.OUT
- net 5.25V: now also C4.1, IC1.EN, IC1.VIN
- net AREF: no longer JP2.3
- net GND: now also C4.2, IC1.GND, IC1.NC; no longer JP1.1, JP2.1
Other:
- note added: "Dynext v2.0 - Arduino-compatible https://github.com/Xevel/dynext"
- note added: "TODO SWD connections, ISP, .. + smaller package"
- note removed: "Dynext v1.0 https://github.com/Xevel/dynext"
- note removed: "Pin for half-duplex from http://asf.atmel.com/docs/3.7.2/xmega.drivers.usart.example3.xmega_e5_xplained/html/index.html"
- moved on the sheet: C14, C6, JP3, JP4, JP5, JP6, JP7, JP8, P1, P2, U2

Commit message: Schematics stabilized, routing in half-way done.
Parts:
- removed F2: TODO, OPL:FUSE-1206
- added C7: 0.1uF, Xevelabs:C0201
- added L2: ferrite, Xevelabs:L0402
- added P5: PIN_SMD_0.8X2, Xevelabs:PIN_SMD_0.8X2
- added P6, P7: PIN_SMD_1X1, Xevelabs:PIN_SMD_1X1
- added R10, R7, R8, R9: 10K, Xevelabs:R0201
- added R6: 47k, Xevelabs:R0201
- JP1: value (none) -> M02PTH; device SparkFun-Connectors:M03PTH -> SparkFun-Connectors:M02PTH
- P1: value PIN_SMD_2X2.5 -> PIN_SMD_0.8X2; device Xevelabs:PIN_SMD_2X2.5 -> Xevelabs:PIN_SMD_0.8X2
- P2: value PIN_SMD_2X2.5 -> PIN_SMD_1X1; device Xevelabs:PIN_SMD_2X2.5 -> Xevelabs:PIN_SMD_1X1
- R1: device Xevelabs:R0402 -> Xevelabs:R0201
- R4: device Xevelabs:R_2-0402 -> Xevelabs:R0201
- U1: value (none) -> TPS62160DSG
- U4: value TXB0101DCK -> TXB0101DRL; device MWquad_stuff:TXB0101DCK -> Xevelabs:TXB0101DRL
Connections:
- removed net D13/LED: R1.2
- removed net DATA_RX: P3.1, U6.PIO0_12/RXD
- removed net DATA_TX: P4.1, U6.PIO0_13/TXD
- removed net MISO: U6.TDI/PIO0_6/AD0, U6.TMS/PIO0_7/AD1
- removed net N$13: U3.AVCC
- removed net N$7: D1.C, D3.A, RPTC1.1, U4.B
- removed net PD0: P1.1
- removed net PD1: P2.1
- removed net SSEL/ISP: U6.PIO0_1/RXD/CLKOUT, U6.PIO0_16/ATRG0/ACMP_I3
- removed net UART0: U4.A
- new net A0: JP6.3, U3.PC0(ADC0/PCINT8)
- new net A1: JP6.4, U3.PC1(ADC1/PCINT9)
- new net A2: JP6.5, U3.PC2(ADC2/PCINT10)
- new net A3: JP6.6, U3.PC3(ADC3/PCINT11)
- new net A4: JP6.7, U3.PC4(ADC4/SDA/PCINT12)
- new net A5: JP5.4, U3.PC5(ADC5/SCL/PCINT13)
- new net ARDU_RST: JP5.2, U3.PC6(!RESET!/PCINT14)
- new net AVCC: C7.2, L2.2, U3.AVCC
- new net D0: JP4.7, U3.PD0(RXD/PCINT16)
- new net D1: JP4.6, U3.PD1(TXD/PCINT17)
- new net D10: JP6.2, U3.PB2(OC1B/SS/PCINT2)
- new net D11: JP4.3, R7.1, U3.PB3(MOSI/OC2A/PCINT3)
- new net D13: JP4.1, R9.1, U3.PB5(SCK/PCINT5)
- new net D2: JP4.5, U3.PD2(INT0/PCINT18)
- new net D3: JP4.4, U3.PD3(INT1/OC2B/PCINT19)
- new net D6(LED): R1.2, U3.PD6(AIN0/OC0A/PCINT22)
- new net D9: JP6.1, U3.PB1(OC1A/PCINT1)
- new net LPC_INT: P6.1, U3.PB0(ICP1/CLKO/PCINT0), U6.PIO0_17/ATRG1/ACMP_I4
- new net LPC_RX: D1.C, D3.A, P5.1, RPTC1.1, U4.B, U6.PIO0_12/RXD
- new net LPC_TX: P4.1, U4.A, U6.PIO0_13/TXD
- new net MISO/D12: JP4.2, U3.PB4(MISO/PCINT4), U6.TDI/PIO0_6/AD0, U6.TMS/PIO0_7/AD1
- new net N$1: P7.1, U6.!TRST!/PIO0_9/AD3
- new net SSEL/ISP/D5: P3.1, U3.PD5(T1/OC0B/PCINT21), U6.PIO0_1/RXD/CLKOUT, U6.PIO0_16/ATRG0/ACMP_I3
- new net TX_EN: P2.1, U4.OE, U6.PIO0_15/TXD/AD7
- net +3V3: now also JP3.4, R4.1, R6.2; no longer R4.1.2, R4.2.2, U4.OE
- net +5V: now also JP3.2, JP7.3, JP7.4, JP7.5, JP7.6, JP7.7, L2.1
- net 5.25V: now also JP1.1, JP7.1, JP7.2
- net AREF: now also JP5.3
- net GND: now also C7.1, JP1.2, JP3.1, JP3.3, JP5.1, JP8.1, JP8.2, JP8.3, JP8.4, JP8.5, JP8.6, JP8.7, P1.1, R10.2, R8.2
- net LPC_RST: now also JP10.4
- net MOSI: now also R7.2, R8.1
- net N$10: now also U3.PB7(TOSC2/XTAL2/PCINT7); no longer U3.PB7
- net N$9: now also U3.PB6(TOSC1/XTAL1/PCINT6); no longer U3.PB6
- net SCK: now also R10.1, R9.2
- net SWCLK: now also JP10.2, R6.1; no longer R4.2.1
- net SWDIO: now also JP10.3, R4.2; no longer R4.1.1
Other:
- note added: "Connectors"
- note added: "LPC_INT : Interrupt pin to signal stuff has changed to the atmega"
- note added: "Level convertion for SPI"
- note added: "Optional short between resets?"
- note added: "TODO LED 0402?"
- note added: "TODO do we put a fuse? what value then? on which rail?"
- note added: "TODO select value"
- note added: "TX_EN : Enable TX level converter or not - also useful to make ISP prog possible"
- note removed: "Expansion connectors"
- note removed: "TODO AVCC using vref or filtered +5V ?"
- note removed: "TODO ISP entry (on B2/SSEL/PIO01) should be accessible for unbricking but also TXD and RXD so that the bootloader could be used..."
- note removed: "TODO SWD connections, ISP, .."
- note removed: "TODO SWD connections, ISP, .. + smaller package"
- note removed: "TODO power led?"
- moved on the sheet: C1, C14, C2, C4, C5, D1, D3, IC1, JP10, JP3, JP4, JP5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

Commit message: Routing is getting close to something viable. I probably will rip up some of the most complex parts to simplifiy them ><
Parts:
- U4: value TXB0101DRL -> TXB0101DCK; device Xevelabs:TXB0101DRL -> Xevelabs:TXB0101DCK
Connections:
- net +3V3: now also JP3.2; no longer JP3.4
- net +5V: now also JP3.4; no longer JP3.2
- net GND: no longer IC1.NC
Changed lines of the file:
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@@
 <grid distance="0.1" unitdist="inch" unit="inch" style="lines" multiple="1" display="no" altdistance="0.01" altunitdist="inch" altunit="inch"/>
 <layers>
-<layer number="1" name="Top" color="4" fill="1" visible="yes" active="no"/>
-<layer number="2" name="Route2" color="1" fill="5" visible="yes" active="no"/>
-<layer number="3" name="Route3" color="4" fill="15" visible="yes" active="no"/>
-<layer number="14" name="Route14" color="1" fill="6" visible="yes" active="no"/>
-<layer number="15" name="Route15" color="4" fill="6" visible="yes" active="no"/>
-<layer number="16" name="Bottom" color="1" fill="1" visible="yes" active="no"/>
-<layer number="17" name="Pads" color="2" fill="1" visible="yes" active="no"/>
-<layer number="18" name="Vias" color="2" fill="1" visible="yes" active="no"/>
-<layer number="19" name="Unrouted" color="6" fill="1" visible="yes" active="no"/>
-<layer number="20" name="Dimension" color="15" fill="1" visible="yes" active="no"/>
-<layer number="21" name="tPlace" color="7" fill="1" visible="yes" active="no"/>
-<layer number="22" name="bPlace" color="7" fill="1" visible="yes" active="no"/>
-<layer number="23" name="tOrigins" color="15" fill="1" visible="yes" active="no"/>
-<layer number="24" name="bOrigins" color="15" fill="1" visible="yes" active="no"/>
-<layer number="25" name="tNames" color="7" fill="1" visible="yes" active="no"/>
-<layer number="26" name="bNames" color="7" fill="1" visible="yes" active="no"/>
-<layer number="27" name="tValues" color="7" fill="1" visible="yes" active="no"/>
-<layer number="28" name="bValues" color="7" fill="1" visible="yes" active="no"/>
+<layer number="1" name="Top" color="4" fill="1" visible="no" active="no"/>
+<layer number="2" name="Route2" color="1" fill="5" visible="no" active="no"/>
+<layer number="3" name="Route3" color="4" fill="15" visible="no" active="no"/>
+<layer number="14" name="Route14" color="1" fill="6" visible="no" active="no"/>
+<layer number="15" name="Route15" color="4" fill="6" visible="no" active="no"/>
+<layer number="16" name="Bottom" color="1" fill="1" visible="no" active="no"/>
+<layer number="17" name="Pads" color="2" fill="1" visible="no" active="no"/>
+<layer number="18" name="Vias" color="2" fill="1" visible="no" active="no"/>
+<layer number="19" name="Unrouted" color="6" fill="1" visible="no" active="no"/>
+<layer number="20" name="Dimension" color="15" fill="1" visible="no" active="no"/>
+<layer number="21" name="tPlace" color="7" fill="1" visible="no" active="no"/>
+<layer number="22" name="bPlace" color="7" fill="1" visible="no" active="no"/>
+<layer number="23" name="tOrigins" color="15" fill="1" visible="no" active="no"/>
+<layer number="24" name="bOrigins" color="15" fill="1" visible="no" active="no"/>
+<layer number="25" name="tNames" color="7" fill="1" visible="no" active="no"/>
+<layer number="26" name="bNames" color="7" fill="1" visible="no" active="no"/>
+<layer number="27" name="tValues" color="7" fill="1" visible="no" active="no"/>
+<layer number="28" name="bValues" color="7" fill="1" visible="no" active="no"/>
 <layer number="29" name="tStop" color="7" fill="3" visible="no" active="no"/>
 <layer number="30" name="bStop" color="7" fill="6" visible="no" active="no"/>
@@
 <layer number="35" name="tGlue" color="7" fill="4" visible="no" active="no"/>
 <layer number="36" name="bGlue" color="7" fill="5" visible="no" active="no"/>
-<layer number="37" name="tTest" color="7" fill="1" visible="yes" active="no"/>
-<layer number="38" name="bTest" color="7" fill="1" visible="yes" active="no"/>
+<layer number="37" name="tTest" color="7" fill="1" visible="no" active="no"/>
+<layer number="38" name="bTest" color="7" fill="1" visible="no" active="no"/>
 <layer number="39" name="tKeepout" color="4" fill="11" visible="no" active="no"/>
 <layer number="40" name="bKeepout" color="1" fill="11" visible="no" active="no"/>
@@
 <layer number="44" name="Drills" color="7" fill="1" visible="no" active="no"/>
 <layer number="45" name="Holes" color="7" fill="1" visible="no" active="no"/>
-<layer number="46" name="Milling" color="3" fill="1" visible="yes" active="no"/>
-<layer number="47" name="Measures" color="7" fill="1" visible="yes" active="no"/>
-<layer number="48" name="Document" color="7" fill="1" visible="yes" active="no"/>
-<layer number="49" name="Reference" color="7" fill="1" visible="yes" active="no"/>
-<layer number="50" name="dxf" color="7" fill="1" visible="yes" active="no"/>
-<layer number="51" name="tDocu" color="7" fill="1" visible="yes" active="no"/>
-<layer number="52" name="bDocu" color="7" fill="1" visible="yes" active="no"/>
-<layer number="53" name="tGND_GNDA" color="7" fill="9" visible="yes" active="no"/>
-<layer number="54" name="bGND_GNDA" color="1" fill="9" visible="yes" active="no"/>
-<layer number="56" name="wert" color="7" fill="1" visible="yes" active="no"/>
+<layer number="46" name="Milling" color="3" fill="1" visible="no" active="no"/>
+<layer number="47" name="Measures" color="7" fill="1" visible="no" active="no"/>
+<layer number="48" name="Document" color="7" fill="1" visible="no" active="no"/>
+<layer number="49" name="Reference" color="7" fill="1" visible="no" active="no"/>
+<layer number="50" name="dxf" color="7" fill="1" visible="no" active="no"/>
+<layer number="51" name="tDocu" color="7" fill="1" visible="no" active="no"/>
+<layer number="52" name="bDocu" color="7" fill="1" visible="no" active="no"/>
+<layer number="53" name="tGND_GNDA" color="7" fill="9" visible="no" active="no"/>
+<layer number="54" name="bGND_GNDA" color="1" fill="9" visible="no" active="no"/>
+<layer number="56" name="wert" color="7" fill="1" visible="no" active="no"/>
 <layer number="91" name="Nets" color="2" fill="1" visible="yes" active="yes"/>
 <layer number="92" name="Busses" color="1" fill="1" visible="yes" active="yes"/>
@@
 <part name="GND17" library="supply1" deviceset="GND" device=""/>
 <part name="D2" library="Xevelabs" deviceset="DIODE" device="-SMP" value="SMP15A-M3/84A"/>
-<part name="U4" library="Xevelabs" deviceset="TXB0101" device="DRL"/>
+<part name="U4" library="Xevelabs" deviceset="TXB0101" device="DCK" value="TXB0101DCK"/>
 <part name="GND18" library="supply1" deviceset="GND" device=""/>
 <part name="P+2" library="supply1" deviceset="+5V" device=""/>
@@
 <instance part="GND29" gate="1" x="210.82" y="198.12" rot="MR0"/>
 <instance part="P7" gate="G$1" x="12.7" y="71.12" rot="R180"/>
-<instance part="P+10" gate="1" x="210.82" y="220.98"/>
-<instance part="+3V7" gate="G$1" x="220.98" y="220.98"/>
+<instance part="P+10" gate="1" x="220.98" y="220.98"/>
+<instance part="+3V7" gate="G$1" x="210.82" y="220.98"/>
 </instances>
 <busses>
@@
 <wire x1="96.52" y1="314.96" x2="99.06" y2="314.96" width="0.1524" layer="91"/>
 <junction x="96.52" y="309.88"/>
-</segment>
-<segment>
-<pinref part="IC1" gate="A" pin="NC"/>
-<wire x1="73.66" y1="309.88" x2="76.2" y2="309.88" width="0.1524" layer="91"/>
-<pinref part="GND7" gate="1" pin="GND"/>
-<wire x1="76.2" y1="304.8" x2="76.2" y2="309.88" width="0.1524" layer="91"/>
 </segment>
 <segment>
@@
 </segment>
 <segment>
-<pinref part="JP3" gate="G$1" pin="4"/>
-<wire x1="215.9" y1="213.36" x2="220.98" y2="213.36" width="0.1524" layer="91"/>
-<wire x1="220.98" y1="213.36" x2="220.98" y2="218.44" width="0.1524" layer="91"/>
 <pinref part="+3V7" gate="G$1" pin="+3V3"/>
+<pinref part="JP3" gate="G$1" pin="2"/>
+<wire x1="210.82" y1="218.44" x2="210.82" y2="213.36" width="0.1524" layer="91"/>
 </segment>
 </net>
@@
 </segment>
 <segment>
-<pinref part="JP3" gate="G$1" pin="2"/>
-<wire x1="210.82" y1="213.36" x2="210.82" y2="218.44" width="0.1524" layer="91"/>
+<pinref part="JP3" gate="G$1" pin="4"/>
+<wire x1="215.9" y1="213.36" x2="220.98" y2="213.36" width="0.1524" layer="91"/>
 <pinref part="P+10" gate="1" pin="+5V"/>
+<wire x1="220.98" y1="213.36" x2="220.98" y2="218.44" width="0.1524" layer="91"/>
 </segment>
 </net>

Commit message: Routing roughly done and seems OK. More verif and silkscreen still needed.
Parts:
- removed JP1: M02PTH, SparkFun-Connectors:M02PTH
Connections:
- net 5.25V: no longer JP1.1
- net GND: no longer JP1.2
Changed lines of the file:
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@@
 <part name="GND20" library="supply1" deviceset="GND" device=""/>
 <part name="GND21" library="supply1" deviceset="GND" device=""/>
-<part name="JP1" library="SparkFun-Connectors" deviceset="M02" device="PTH"/>
-<part name="GND27" library="supply1" deviceset="GND" device=""/>
 <part name="C4" library="Xevelabs" deviceset="C" device="0402" value="1uF"/>
 <part name="GND28" library="supply1" deviceset="GND" device=""/>
@@
 <instance part="GND20" gate="1" x="45.72" y="350.52"/>
 <instance part="GND21" gate="1" x="35.56" y="350.52"/>
-<instance part="JP1" gate="G$1" x="210.82" y="167.64" rot="MR270"/>
-<instance part="GND27" gate="1" x="208.28" y="157.48" rot="MR0"/>
 <instance part="C4" gate="G$1" x="25.4" y="312.42"/>
 <instance part="GND28" gate="1" x="25.4" y="302.26"/>
@@
 </segment>
 <segment>
-<pinref part="GND27" gate="1" pin="GND"/>
-<pinref part="JP1" gate="G$1" pin="2"/>
-</segment>
-<segment>
 <pinref part="C4" gate="G$1" pin="2"/>
 <wire x1="25.4" y1="304.8" x2="25.4" y2="309.88" width="0.1524" layer="91"/>
@@
 <junction x="269.24" y="175.26"/>
 </segment>
-<segment>
-<pinref part="JP1" gate="G$1" pin="1"/>
-<wire x1="210.82" y1="160.02" x2="220.98" y2="160.02" width="0.1524" layer="91"/>
-<label x="220.98" y="167.64" size="1.778" layer="95"/>
-<wire x1="220.98" y1="160.02" x2="220.98" y2="167.64" width="0.1524" layer="91"/>
-</segment>
-</net>
+</net>

Commit message: Added all the silkscreen. Potentially ready.
Parts:
- JP3, JP5: device SparkFun-Connectors:M04PTH -> SparkFun-Connectors:M041X04_NO_SILK
- JP4, JP6, JP7: device SparkFun-Connectors:M07 -> Xevelabs:M07NO_SILK
- JP8: device SparkFun-Connectors:M07 -> Xevelabs:M07SQUARE_ALL
- U6: value LPC11A02UK,118 -> IC_LPC11A0UK,118; device Xevelabs:LPC11A02UK,118 -> Xevelabs:IC_LPC11A0UK,118
Changed lines of the file:
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@@
 <grid distance="0.1" unitdist="inch" unit="inch" style="lines" multiple="1" display="no" altdistance="0.01" altunitdist="inch" altunit="inch"/>
 <layers>
-<layer number="1" name="Top" color="4" fill="1" visible="no" active="no"/>
-<layer number="2" name="Route2" color="1" fill="5" visible="no" active="no"/>
-<layer number="3" name="Route3" color="4" fill="15" visible="no" active="no"/>
-<layer number="14" name="Route14" color="1" fill="6" visible="no" active="no"/>
-<layer number="15" name="Route15" color="4" fill="6" visible="no" active="no"/>
-<layer number="16" name="Bottom" color="1" fill="1" visible="no" active="no"/>
-<layer number="17" name="Pads" color="2" fill="1" visible="no" active="no"/>
-<layer number="18" name="Vias" color="2" fill="1" visible="no" active="no"/>
-<layer number="19" name="Unrouted" color="6" fill="1" visible="no" active="no"/>
-<layer number="20" name="Dimension" color="15" fill="1" visible="no" active="no"/>
-<layer number="21" name="tPlace" color="7" fill="1" visible="no" active="no"/>
-<layer number="22" name="bPlace" color="7" fill="1" visible="no" active="no"/>
-<layer number="23" name="tOrigins" color="15" fill="1" visible="no" active="no"/>
-<layer number="24" name="bOrigins" color="15" fill="1" visible="no" active="no"/>
-<layer number="25" name="tNames" color="7" fill="1" visible="no" active="no"/>
-<layer number="26" name="bNames" color="7" fill="1" visible="no" active="no"/>
-<layer number="27" name="tValues" color="7" fill="1" visible="no" active="no"/>
-<layer number="28" name="bValues" color="7" fill="1" visible="no" active="no"/>
+<layer number="1" name="Top" color="4" fill="1" visible="yes" active="no"/>
+<layer number="2" name="Route2" color="1" fill="5" visible="yes" active="no"/>
+<layer number="3" name="Route3" color="4" fill="15" visible="yes" active="no"/>
+<layer number="14" name="Route14" color="1" fill="6" visible="yes" active="no"/>
+<layer number="15" name="Route15" color="4" fill="6" visible="yes" active="no"/>
+<layer number="16" name="Bottom" color="1" fill="1" visible="yes" active="no"/>
+<layer number="17" name="Pads" color="2" fill="1" visible="yes" active="no"/>
+<layer number="18" name="Vias" color="2" fill="1" visible="yes" active="no"/>
+<layer number="19" name="Unrouted" color="6" fill="1" visible="yes" active="no"/>
+<layer number="20" name="Dimension" color="15" fill="1" visible="yes" active="no"/>
+<layer number="21" name="tPlace" color="7" fill="1" visible="yes" active="no"/>
+<layer number="22" name="bPlace" color="7" fill="1" visible="yes" active="no"/>
+<layer number="23" name="tOrigins" color="15" fill="1" visible="yes" active="no"/>
+<layer number="24" name="bOrigins" color="15" fill="1" visible="yes" active="no"/>
+<layer number="25" name="tNames" color="7" fill="1" visible="yes" active="no"/>
+<layer number="26" name="bNames" color="7" fill="1" visible="yes" active="no"/>
+<layer number="27" name="tValues" color="7" fill="1" visible="yes" active="no"/>
+<layer number="28" name="bValues" color="7" fill="1" visible="yes" active="no"/>
 <layer number="29" name="tStop" color="7" fill="3" visible="no" active="no"/>
 <layer number="30" name="bStop" color="7" fill="6" visible="no" active="no"/>
@@
 <layer number="35" name="tGlue" color="7" fill="4" visible="no" active="no"/>
 <layer number="36" name="bGlue" color="7" fill="5" visible="no" active="no"/>
-<layer number="37" name="tTest" color="7" fill="1" visible="no" active="no"/>
-<layer number="38" name="bTest" color="7" fill="1" visible="no" active="no"/>
+<layer number="37" name="tTest" color="7" fill="1" visible="yes" active="no"/>
+<layer number="38" name="bTest" color="7" fill="1" visible="yes" active="no"/>
 <layer number="39" name="tKeepout" color="4" fill="11" visible="no" active="no"/>
 <layer number="40" name="bKeepout" color="1" fill="11" visible="no" active="no"/>
@@
 <layer number="44" name="Drills" color="7" fill="1" visible="no" active="no"/>
 <layer number="45" name="Holes" color="7" fill="1" visible="no" active="no"/>
-<layer number="46" name="Milling" color="3" fill="1" visible="no" active="no"/>
-<layer number="47" name="Measures" color="7" fill="1" visible="no" active="no"/>
-<layer number="48" name="Document" color="7" fill="1" visible="no" active="no"/>
-<layer number="49" name="Reference" color="7" fill="1" visible="no" active="no"/>
-<layer number="50" name="dxf" color="7" fill="1" visible="no" active="no"/>
-<layer number="51" name="tDocu" color="7" fill="1" visible="no" active="no"/>
-<layer number="52" name="bDocu" color="7" fill="1" visible="no" active="no"/>
-<layer number="53" name="tGND_GNDA" color="7" fill="9" visible="no" active="no"/>
-<layer number="54" name="bGND_GNDA" color="1" fill="9" visible="no" active="no"/>
-<layer number="56" name="wert" color="7" fill="1" visible="no" active="no"/>
+<layer number="46" name="Milling" color="3" fill="1" visible="yes" active="no"/>
+<layer number="47" name="Measures" color="7" fill="1" visible="yes" active="no"/>
+<layer number="48" name="Document" color="7" fill="1" visible="yes" active="no"/>
+<layer number="49" name="Reference" color="7" fill="1" visible="yes" active="no"/>
+<layer number="50" name="dxf" color="7" fill="1" visible="yes" active="no"/>
+<layer number="51" name="tDocu" color="7" fill="1" visible="yes" active="no"/>
+<layer number="52" name="bDocu" color="7" fill="1" visible="yes" active="no"/>
+<layer number="53" name="tGND_GNDA" color="7" fill="9" visible="yes" active="no"/>
+<layer number="54" name="bGND_GNDA" color="1" fill="9" visible="yes" active="no"/>
+<layer number="56" name="wert" color="7" fill="1" visible="yes" active="no"/>
 <layer number="91" name="Nets" color="2" fill="1" visible="yes" active="yes"/>
 <layer number="92" name="Busses" color="1" fill="1" visible="yes" active="yes"/>
@@
 <part name="R1" library="Xevelabs" deviceset="R" device="0201" value="1K"/>
 <part name="+3V2" library="supply1" deviceset="+3V3" device=""/>
-<part name="JP3" library="SparkFun-Connectors" deviceset="M04" device="PTH"/>
-<part name="JP4" library="SparkFun-Connectors" deviceset="M07" device=""/>
-<part name="JP5" library="SparkFun-Connectors" deviceset="M04" device="PTH"/>
-<part name="JP6" library="SparkFun-Connectors" deviceset="M07" device=""/>
-<part name="JP7" library="SparkFun-Connectors" deviceset="M07" device=""/>
-<part name="JP8" library="SparkFun-Connectors" deviceset="M07" device=""/>
-<part name="U6" library="Xevelabs" deviceset="LPC11A02UK,118" device=""/>
+<part name="JP3" library="SparkFun-Connectors" deviceset="M04" device="1X04_NO_SILK"/>
+<part name="JP4" library="Xevelabs" deviceset="M07" device="NO_SILK"/>
+<part name="JP5" library="SparkFun-Connectors" deviceset="M04" device="1X04_NO_SILK"/>
+<part name="JP6" library="Xevelabs" deviceset="M07" device="NO_SILK"/>
+<part name="JP7" library="Xevelabs" deviceset="M07" device="NO_SILK"/>
+<part name="JP8" library="Xevelabs" deviceset="M07" device="SQUARE_ALL"/>
+<part name="U6" library="Xevelabs" deviceset="IC_LPC11A0?UK,118" device=""/>
 <part name="GND5" library="supply1" deviceset="GND" device=""/>
 <part name="JP10" library="SparkFun-Connectors" deviceset="M05" device="1.27MM" value="SWD"/>

Commit message: Rearrangement of the schematics for better fitting on the screen
Connections:
- net N$1 renamed TEST_POINT
Other:
- note removed: "Optional short between resets?"
- moved on the sheet: C1, C13, C14, C17, C2, C3, C4, C5, C6, C7, D1, D2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
